Commit message: Autonavigation

File: src/drone_simulation/urdf/rescue_drone.urdf.xacro (robot description, xacro)
@@ -5,26 +5,50 @@
     <color rgba="0.0 0.0 0.0 1.0"/>
   </material>
-  <material name="grey">
-    <color rgba="0.5 0.5 0.5 1.0"/>
+  <material name="orange">
+    <color rgba="1.0 0.5 0.0 1.0"/>
   </material>
   <!-- Base Link (Body) -->
   <link name="base_link">
     <inertial>
-      <mass value="1.0"/>
+      <mass value="0.8"/>
       <origin xyz="0 0 0" rpy="0 0 0"/>
-      <inertia ixx="0.01" ixy="0" ixz="0" iyy="0.01" iyz="0" izz="0.02"/>
+      <inertia ixx="0.005" ixy="0" ixz="0" iyy="0.005" iyz="0" izz="0.01"/>
     </inertial>
     <visual>
       <geometry>
-        <box size="0.3 0.3 0.1"/>
-      </geometry>
-      <material name="grey"/>
+        <box size="0.2 0.2 0.07"/>
+      </geometry>
+      <material name="orange"/>
     </visual>
     <collision>
       <geometry>
-        <box size="0.3 0.3 0.1"/>
+        <box size="0.2 0.2 0.07"/>
       </geometry>
     </collision>
   </link>
+  <!-- Gazebo Material for Base Link and Bumper -->
+  <gazebo reference="base_link">
+    <visual>
+      <material>
+        <ambient>1.0 0.5 0.0 1.0</ambient>
+        <diffuse>1.0 0.5 0.0 1.0</diffuse>
+        <specular>0.1 0.1 0.1 1.0</specular>
+        <emissive>0.0 0.0 0.0 0.0</emissive>
+      </material>
+    </visual>
+    <sensor name="drone_bumper" type="contact">
+      <always_on>true</always_on>
+      <update_rate>50.0</update_rate>
+      <contact>
+        <collision>base_link_collision</collision>
+      </contact>
+      <plugin name="drone_bumper_plugin" filename="libgazebo_ros_bumper.so">
+        <ros>
+          <remapping>bumper_states:=/drone/collisions</remapping>
+        </ros>
+        <frame_name>base_link</frame_name>
+      </plugin>
+    </sensor>
+  </gazebo>
   <!-- Gazebo ROS State Plugin -->
   <gazebo>
@@ -45,17 +69,38 @@
   </gazebo>
   <!-- Sensors -->
-  <!-- Camera -->
-  <link name="camera_link">
-    <visual>
-      <geometry>
-        <box size="0.05 0.05 0.05"/>
-      </geometry>
-      <material name="black"/>
-    </visual>
-  </link>
+  <!-- Stereo Camera Base -->
+  <link name="camera_link"/>
   <joint name="camera_joint" type="fixed">
     <parent link="base_link"/>
     <child link="camera_link"/>
-    <origin xyz="0.15 0 0.05" rpy="0 0 0"/>
+    <origin xyz="0.1 0 0.035" rpy="0 0 0"/>
+  </joint>
+  <!-- Left Camera -->
+  <link name="camera_left_link">
+    <visual>
+      <geometry>
+        <box size="0.02 0.02 0.02"/>
+      </geometry>
+      <material name="black"/>
+    </visual>
+  </link>
+  <joint name="camera_left_joint" type="fixed">
+    <parent link="camera_link"/>
+    <child link="camera_left_link"/>
+    <origin xyz="0 0.03 0" rpy="0 0 0"/>
+  </joint>
+  <!-- Right Camera -->
+  <link name="camera_right_link">
+    <visual>
+      <geometry>
+        <box size="0.02 0.02 0.02"/>
+      </geometry>
+      <material name="black"/>
+    </visual>
+  </link>
+  <joint name="camera_right_joint" type="fixed">
+    <parent link="camera_link"/>
+    <child link="camera_right_link"/>
+    <origin xyz="0 -0.03 0" rpy="0 0 0"/>
   </joint>
   <!-- IMU -->
@@ -78,5 +123,5 @@
     <parent link="base_link"/>
     <child link="dtof_link"/>
-    <origin xyz="0.15 0 -0.02" rpy="0 0 0"/>
+    <origin xyz="0.1 0 -0.01" rpy="0 0 0"/>
   </joint>
   <!-- dToF Back (Range) -->
@@ -92,11 +137,12 @@
     <parent link="base_link"/>
     <child link="dtof_back_link"/>
-    <origin xyz="-0.15 0 -0.02" rpy="0 0 3.14159"/>
+    <origin xyz="-0.1 0 -0.01" rpy="0 0 3.14159"/>
   </joint>
   <!-- Gazebo Plugins for Sensors -->
-  <gazebo reference="camera_link">
-    <sensor type="camera" name="rgb_camera">
+  <!-- Left Camera -->
+  <gazebo reference="camera_left_link">
+    <sensor type="camera" name="left_camera">
       <update_rate>30.0</update_rate>
-      <camera name="head">
+      <camera name="left">
         <horizontal_fov>1.3962634</horizontal_fov>
         <image>
@@ -110,10 +156,38 @@
         </clip>
       </camera>
-      <plugin name="camera_controller" filename="libgazebo_ros_camera.so">
-        <ros>
-          <remapping>image_raw:=/camera/image_raw</remapping>
-          <remapping>camera_info:=/camera/camera_info</remapping>
-        </ros>
-        <frame_name>camera_link</frame_name>
+      <plugin name="left_camera_controller" filename="libgazebo_ros_camera.so">
+        <ros>
+          <remapping>image_raw:=/left/image_raw</remapping>
+          <remapping>camera_info:=/left/camera_info</remapping>
+        </ros>
+        <camera_name>left</camera_name>
+        <frame_name>camera_left_link</frame_name>
+      </plugin>
+    </sensor>
+  </gazebo>
+  <!-- Right Camera -->
+  <gazebo reference="camera_right_link">
+    <sensor type="camera" name="right_camera">
+      <update_rate>30.0</update_rate>
+      <camera name="right">
+        <horizontal_fov>1.3962634</horizontal_fov>
+        <image>
+          <width>800</width>
+          <height>600</height>
+          <format>R8G8B8</format>
+        </image>
+        <clip>
+          <near>0.02</near>
+          <far>300</far>
+        </clip>
+      </camera>
+      <plugin name="right_camera_controller" filename="libgazebo_ros_camera.so">
+        <ros>
+          <remapping>image_raw:=/right/image_raw</remapping>
+          <remapping>camera_info:=/right/camera_info</remapping>
+        </ros>
+        <camera_name>right</camera_name>
+        <frame_name>camera_right_link</frame_name>
+        <hack_baseline>0.06</hack_baseline>
       </plugin>
     </sensor>

Commit message: Update

File: src/drone_simulation/urdf/rescue_drone.urdf.xacro (robot description, xacro)
@@ -51,13 +51,17 @@
     </sensor>
   </gazebo>
-  <!-- Gazebo ROS State Plugin -->
-  <gazebo>
-    <plugin name="gazebo_ros_state" filename="libgazebo_ros_state.so"/>
-  </gazebo>
-  <!-- Simple Movement Plugin -->
+  <!-- Dummy root link to fix KDL warning and improve stability -->
+  <link name="base_footprint"/>
+  <joint name="base_joint" type="fixed">
+    <parent link="base_footprint"/>
+    <child link="base_link"/>
+    <origin xyz="0 0 0" rpy="0 0 0"/>
+  </joint>
+  <!-- Movement Plugin -->
   <gazebo>
     <plugin name="drone_move_controller" filename="libgazebo_ros_planar_move.so">
       <ros>
         <remapping>cmd_vel:=/cmd_vel</remapping>
+        <remapping>odom:=/odom</remapping>
       </ros>
       <update_rate>50</update_rate>
@@ -65,5 +69,5 @@
       <publish_odom_tf>true</publish_odom_tf>
       <odometry_frame>odom</odometry_frame>
-      <robot_base_frame>base_link</robot_base_frame>
+      <robot_base_frame>base_footprint</robot_base_frame>
     </plugin>
   </gazebo>
