Commit message: update

File: src/drone_simulation/urdf/rescue_drone.urdf.xacro (robot description, xacro)
@@ -21,5 +21,5 @@
       <material name="orange"/>
     </visual>
-    <collision>
+    <collision name="base_link_collision">
       <geometry>
         <box size="0.2 0.2 0.07"/>

Commit message: VAE+LSTM+PPO

File: src/drone_simulation/urdf/rescue_drone.urdf.xacro (robot description, xacro)
@@ -27,6 +27,8 @@
     </collision>
   </link>
-  <!-- Gazebo Material for Base Link and Bumper -->
+  <!-- Gazebo settings for Base Link: visual, bumper sensor, gravity -->
   <gazebo reference="base_link">
+    <material>Gazebo/Grey</material>
+    <gravity>0</gravity>
     <visual>
       <material>
@@ -92,5 +94,5 @@
     <parent link="camera_link"/>
     <child link="camera_left_link"/>
-    <origin xyz="0 0.03 0" rpy="0 0 0"/>
+    <origin xyz="0 0.06 0" rpy="0 0 0"/>
   </joint>
   <!-- Right Camera -->
@@ -106,5 +108,5 @@
     <parent link="camera_link"/>
     <child link="camera_right_link"/>
-    <origin xyz="0 -0.03 0" rpy="0 0 0"/>
+    <origin xyz="0 -0.06 0" rpy="0 0 0"/>
   </joint>
   <!-- IMU -->
@@ -151,6 +153,6 @@
         <horizontal_fov>1.3962634</horizontal_fov>
         <image>
-          <width>800</width>
-          <height>600</height>
+          <width>640</width>
+          <height>480</height>
           <format>R8G8B8</format>
         </image>
@@ -177,6 +179,6 @@
         <horizontal_fov>1.3962634</horizontal_fov>
         <image>
-          <width>800</width>
-          <height>600</height>
+          <width>640</width>
+          <height>480</height>
           <format>R8G8B8</format>
         </image>
@@ -193,5 +195,5 @@
         <camera_name>right</camera_name>
         <frame_name>camera_right_link</frame_name>
-        <hack_baseline>0.06</hack_baseline>
+        <hack_baseline>0.12</hack_baseline>
       </plugin>
     </sensor>
@@ -265,7 +267,3 @@
     </sensor>
   </gazebo>
-  <gazebo reference="base_link">
-    <material>Gazebo/Grey</material>
-    <gravity>0</gravity>
-  </gazebo>
 </robot>
